File: PCB/SmartLed.sch (EAGLE design)
At the start: 51 parts, among them IC2 DS1307, IC3 MEGA8-P, K1 G5LE, Q2 32.768khz, T1 BC337

Commit message: Working on adding battery voltage meter & adding esp8266 connections header
Parts:
- removed JP2: (no value), pinhead:PINHD-1X2
- removed LED-OUT: (no value), con-ptr500:AK500/2
- removed LED3: (no value), led:LED3MM
- added CONTROL-OUT: (no value), con-ptr500:AK500/2
- added IC4: LM1117T(H)-3.3, lm1117_10:LM1117T(H)-3.3
- added R6: 100k, rcl:R-EU_0207/10
- added SV1: (no value), con-lstb:MA04-2
- R8: value 1.2k -> 10k
Connections:
- new net N$18: IC3.PC1(ADC1), R6.2, R8.1
- net +12V: now also R6.1; no longer K12.P
- net GND: now also R8.2; no longer LED-OUT-1.KL, LED3.C
- net N$11: now also IC3.PB5(SCK); no longer IC3.PD0(RXD)
- net N$16: now also CONTROL-OUT-1.KL, K12.O; no longer LED3.A, R8.2
- net N$28: now also IC3.PD2(INT0); no longer IC3.PD1(TXD)
- net N$30: now also IC3.PD1(TXD); no longer IC3.PC1(ADC1), JP2.1
- net N$31: now also IC3.PD5(T1); no longer IC3.PD4(XCK/T0)
- net N$32: now also IC3.PD3(INT1); no longer IC3.PD2(INT0)
- net N$33: now also IC3.PD4(XCK/T0); no longer IC3.PD3(INT1)
- net N$34: now also IC3.PD0(RXD); no longer IC3.PC2(ADC2), JP2.2
- net N$8: now also CONTROL-OUT-2.KL; no longer LED-OUT-2.KL, R8.1
Other:
- moved on the sheet: C5, D1, JP1, K1, LED5, LED6, LED7, LED8, R1, R10, R11, R12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
